File: PicoADXL.kicad_sch (KiCad schematic)
At the start: 35 parts, among them J1 USB_CONN, SW1 SW_Push, SW2 SW_Push, U1 RP2040, U2 ADXL345, U3 WL2803K, U4 W25Q64JVXGIQ, U5 12MHz

Commit message: added lcsc part # field for fab toolkit
Parts:
- C1, C2: LCSC Part # (none) -> C109456
- C10: LCSC Part # (none) -> C107037
- C11, C15: LCSC Part # (none) -> C106214
- C12, C13, C14, C16, C3, C4, C5, C6, C7, C8, C9: LCSC Part # (none) -> C14663
- D1: LCSC Part # (none) -> C434421
- J1: LCSC Part # (none) -> C136657
- R1, R2: LCSC Part # (none) -> C185346
- R3, R4, R5, R7: LCSC Part # (none) -> C98220
- R6: LCSC Part # (none) -> C114617
- R8: LCSC Part # (none) -> C22548
- SW1, SW2: LCSC Part # (none) -> C963349
- U1: LCSC Part # (none) -> C2040; LCSC# C2040 -> C2040
- U2: LCSC Part # (none) -> C9667
- U3: LCSC Part # (none) -> C192927
- U4: LCSC Part # (none) -> C2940195
- U5: LCSC Part # (none) -> C7425459
